Commit message: Model additions
- Modeled 3-constant electric motor
- Created a Skywalker-like aircraft model

File: last_letter/urdf/skywalker_2013.urdf (robot description, URDF)
Before this commit: robot plane, 1 links, 0 joints
Links:
- link base_link: geometry visual mesh filename=package://last_letter/urdf/skywalker_2013.stl scale=0.02621 0.02621 0.02621
