Commit message: Moved 3D model files to aircraft folder
Now they can be found under the `/data/parameters/<aircraft_name>/urdf` folder, instead of `urdf`.
This allows for completely independent aircraft folders.

File: last_letter/data/parameters/aircraft/HCUAV/urdf/HCUAV.urdf (robot description, URDF)
Before this commit: robot plane, 1 links, 0 joints
Links:
- link base_link: geometry visual mesh filename=package://last_letter/data/parameters/aircraft/HCUAV/urdf/H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 scale=0.0256 0.0256 0.0256

File: last_letter/data/parameters/aircraft/skywalker_2013/urdf/skywalker_2013.urdf (robot description, URDF)
Before this commit: robot plane, 1 links, 0 joints
Links:
- link base_link: geometry visual mesh filename=package://last_letter/data/parameters/aircraft/skywalker_20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 scale=0.02621 0.02621 0.02621
