Commit message: First jab at thrust vectoring
Temporarilly, the skywalker_2013 model has a configuration where the propeller is gimballed on the pitch axis using the rudder channel.

Thrust vectoring is the first step towards hybrid vehicles and multicopter modelling.

Over the next commints this functionality will be migrated into a dedicated vehicle model/folder.

File: last_letter/data/parameters/aircraft/skywalker_2013/urdf/skywalker_2013.urdf (robot description, URDF)
Before this commit: robot plane, 1 links, 0 joints
Links:
- added link propeller; visual mesh filename=package://last_letter/data/parameters/aircraft/skywalker_20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
Joints:
- added joint motor_mount: type floating, parent base_link, child propeller
