Commit message: Created the frist multi-motor aircraft
The firefly_Y6 aircraft folder was created
There are severe issues with the propeller behavious.
Most notably, the torque produced seems VERY excessive.

File: last_letter/data/parameters/aircraft/firefly_Y6/urdf/firefly_Y6.urdf (robot description, URDF)
Before this commit: robot plane, 2 links, 1 joints
Links:
- added link propeller_2; visual mesh filename=package://last_letter/data/parameters/aircraft/firefly_Y6/u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
- added link propeller_3; visual mesh filename=package://last_letter/data/parameters/aircraft/firefly_Y6/u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
Joints:
- removed joint motor_mount
- added joint motor_mount_1: type floating, parent base_link, child propeller_1
- added joint motor_mount_2: type floating, parent base_link, child propeller_2
- added joint motor_mount_3: type floating, parent base_link, child propeller_3

File: last_letter/data/parameters/aircraft/skywalker_2013/urdf/skywalker_2013.urdf (robot description, URDF)
Before this commit: robot plane, 2 links, 1 joints
Links:
- removed link propeller
- added link propeller_1; visual mesh filename=package://last_letter/data/parameters/aircraft/skywalker_20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
Joints:
- joint motor_mount: child propeller -> propeller_1

Commit message: Updates in firefly_Y6 in an effort to make it stable

File: last_letter/data/parameters/aircraft/firefly_Y6/urdf/firefly_Y6.urdf (robot description, URDF)
Before this commit: robot plane, 4 links, 3 joints
Links:
- added link propeller_4; visual mesh filename=package://last_letter/data/parameters/aircraft/firefly_Y6/u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
- added link propeller_5; visual mesh filename=package://last_letter/data/parameters/aircraft/firefly_Y6/u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
- added link propeller_6; visual mesh filename=package://last_letter/data/parameters/aircraft/firefly_Y6/u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
Joints:
- added joint motor_mount_4: type floating, parent base_link, child propeller_4
- added joint motor_mount_5: type floating, parent base_link, child propeller_5
- added joint motor_mount_6: type floating, parent base_link, child propeller_6
